Commit message: config files

File: WarehouseBot/urdf/_d435.gazebo.xacro (robot description, xacro)
@@ -134,4 +134,9 @@
       	<pointCloudTopicName>depth/points</pointCloudTopicName>
       	<pointCloudCutoff>0.5</pointCloudCutoff>
+          <!-- <distortionK1>0</distortionK1>
+          <distortionK2>0</distortionK2>
+          <distortionK3>0</distortionK3>
+          <distortionT1>0</distortionT1>
+          <distortionT2>0</distortionT2> -->
       </plugin>
     </gazebo>

File: WarehouseBot/urdf/warehousebot.xacro (robot description, xacro)
@@ -759,5 +759,5 @@
 -->s
   <!--Please do not delete the below commented code. It will be used when we move the Scissorlift Mechanism-->
-  <joint name="topslider" type="prismatic">
+  <joint name="topslider" type="fixed">
     <origin rpy="0 0 0" xyz="0.32 -0.000187 0.0"/>
     <parent link="scissortop"/>
